Commit message: ddog第一阶段和第二阶段的sim2sim仿真

File: legged_gym/resources/robots/Ddog/urdf/Ddog.urdf (robot description, URDF)
Before this commit: robot hje3, 17 links, 16 joints
Links:
- added link real_sense, mass 0.05; collision box size=0.01 0.1 0.02; visual box size=0.01 0.1 0.02
Joints:
- added joint realsense_joint: type fixed, parent base_link, child real_sense, origin xyz=0.255 0 0.065 rpy=0 0.436 0, axis 0 0 1
